Commit message: broken graph

File: body.urdf (robot description, URDF)
Before this commit: robot robot, 9 links, 8 joints
Links:
- removed link BackLeg
- removed link BackLowerLeg
- removed link FrontLeg
- removed link FrontLowerLeg
- removed link LeftLeg
- removed link LeftLowerLeg
- removed link RightLeg
- removed link RightLowerLeg
- added link BackLeftLeg, mass 1; collision box size=0.2 1 0.2; visual box size=0.2 1 0.2
- added link BackLeftLowerLeg, mass 1; collision box size=0.2 0.2 1; visual box size=0.2 0.2 1
- added link BackRightLeg, mass 1; collision box size=0.2 1 0.2; visual box size=0.2 1 0.2
- added link BackRightLowerLeg, mass 1; collision box size=0.2 0.2 1; visual box size=0.2 0.2 1
- added link FrontLeftLeg, mass 1; collision box size=0.2 1 0.2; visual box size=0.2 1 0.2
- added link FrontLeftLowerLeg, mass 1; collision box size=0.2 0.2 1; visual box size=0.2 0.2 1
- added link FrontRightLeg, mass 1; collision box size=0.2 1 0.2; visual box size=0.2 1 0.2
- added link FrontRightLowerLeg, mass 1; collision box size=0.2 0.2 1; visual box size=0.2 0.2 1
- added link MiddleLeftLeg, mass 1; collision box size=0.2 1 0.2; visual box size=0.2 1 0.2
- added link MiddleLeftLowerLeg, mass 1; collision box size=0.2 0.2 1; visual box size=0.2 0.2 1
- added link MiddleRightLeg, mass 1; collision box size=0.2 1 0.2; visual box size=0.2 1 0.2
- added link MiddleRightLowerLeg, mass 1; collision box size=0.2 0.2 1; visual box size=0.2 0.2 1
- link Torso: geometry collision box size=1.7 1 1; visual box size=1.7 1 1
Joints:
- removed joint BackLeg_BackLowerLeg
- removed joint FrontLeg_FrontLowerLeg
- removed joint LeftLeg_LeftLowerLeg
- removed joint RightLeg_RightLowerLeg
- removed joint Torso_BackLeg
- removed joint Torso_FrontLeg
- removed joint Torso_LeftLeg
- removed joint Torso_RightLeg
- added joint BackLeftLeg_BackLeftLowerLeg: type revolute, parent BackLeftLeg, child BackLeftLowerLeg, origin xyz=-0.3 -1 0 rpy=0 0 0, axis 0 1 0, limit lower=-3.14159 upper=3.14159 effort=0.0 velocity=0.0
- added joint BackRightLeg_BackRightLowerLeg: type revolute, parent BackRightLeg, child BackRightLowerLeg, origin xyz=-0.3 1 0 rpy=0 0 0, axis 0 1 0, limit lower=-3.14159 upper=3.14159 effort=0.0 velocity=0.0
- added joint FrontLeftLeg_FrontLeftLowerLeg: type revolute, parent FrontLeftLeg, child FrontLeftLowerLeg, origin xyz=0.3 -1 0 rpy=0 0 0, axis 1 0 0, limit lower=-3.14159 upper=3.14159 effort=0.0 velocity=0.0
- added joint FrontRightLeg_FrontRightLowerLeg: type revolute, parent FrontRightLeg, child FrontRightLowerLeg, origin xyz=0.3 1 0 rpy=0 0 0, axis 1 0 0, limit lower=-3.14159 upper=3.14159 effort=0.0 velocity=0.0
- added joint MiddleLeftLeg_MiddleLeftLowerLeg: type revolute, parent MiddleLeftLeg, child MiddleLeftLowerLeg, origin xyz=0 -1 0 rpy=0 0 0, axis 0 1 0, limit lower=-3.14159 upper=3.14159 effort=0.0 velocity=0.0
- added joint MiddleRightLeg_MiddleRightLowerLeg: type revolute, parent MiddleRightLeg, child MiddleRightLowerLeg, origin xyz=0 1 0 rpy=0 0 0, axis 0 1 0, limit lower=-3.14159 upper=3.14159 effort=0.0 velocity=0.0
- added joint Torso_BackLeftLeg: type revolute, parent Torso, child BackLeftLeg, origin xyz=-0.3 -0.5 1 rpy=0 0 0, axis 1 0 0, limit lower=-3.14159 upper=3.14159 effort=0.0 velocity=0.0
- added joint Torso_BackRightLeg: type revolute, parent Torso, child BackRightLeg, origin xyz=-0.3 0.5 1 rpy=0 0 0, axis 1 0 0, limit lower=-3.14159 upper=3.14159 effort=0.0 velocity=0.0
- added joint Torso_FrontLeftLeg: type revolute, parent Torso, child FrontLeftLeg, origin xyz=0.3 -0.5 1 rpy=0 0 0, axis 1 0 0, limit lower=-3.14159 upper=3.14159 effort=0.0 velocity=0.0
- added joint Torso_FrontRightLeg: type revolute, parent Torso, child FrontRightLeg, origin xyz=0.3 0.5 1 rpy=0 0 0, axis 1 0 0, limit lower=-3.14159 upper=3.14159 effort=0.0 velocity=0.0
- added joint Torso_MiddleLeftLeg: type revolute, parent Torso, child MiddleLeftLeg, origin xyz=0 -0.5 1 rpy=0 0 0, axis 1 0 0, limit lower=-3.14159 upper=3.14159 effort=0.0 velocity=0.0
- added joint Torso_MiddleRightLeg: type revolute, parent Torso, child MiddleRightLeg, origin xyz=0 0.5 1 rpy=0 0 0, axis 1 0 0, limit lower=-3.14159 upper=3.14159 effort=0.0 velocity=0.0

Commit message: still broken...

File: body.urdf (robot description, URDF)
Before this commit: robot robot, 13 links, 12 joints
Joints:
- joint FrontLeftLeg_FrontLeftLowerLeg: axis 1 0 0 -> 0 1 0
- joint FrontRightLeg_FrontRightLowerLeg: axis 1 0 0 -> 0 1 0

Commit message: fixed graph

File: body.urdf (robot description, URDF)
Before this commit: robot robot, 13 links, 12 joints
Joints:
- joint BackLeftLeg_BackLeftLowerLeg: axis 0 1 0 -> 1 0 0
- joint FrontRightLeg_FrontRightLowerLeg: axis 0 1 0 -> 1 0 0
